File: MicroFLiC_I2C_extension_1_0.kicad_pcb (KiCad board)
At the start: 2 copper layers, 49.8 x 49.8 mm, 13 parts, among them P1 Header_1x14, P2 Socket_1x14, P3 8-188275-4, P4 Header_1x4, P5 Socket_1x4, P6 DB15-VGA, P7 RJ45, SW1 SW_PUSH, SW2 DIPS_04

Commit message: Final production board v1.0
Other:
- board text added: "12V"
- board text added: "2V5"
- board text added: "3V3"
- board text added: "5V"
- board text added: "Reset"
- board text added: "SW1"
- board text added: "SW2"
- board text added: "SW3"
- board text added: "SW4"
