File: MicroFLiC_I2C_extension.sch (KiCad schematic (older format))
At the start: 13 parts, among them P1 Header_1x14, P2 Socket_1x14, P3 Micro-MaTch 14 way, P4 Header_1x4, P5 Socket_1x4, P6 DB15-VGA, P7 RJ45, SW1 SW_PUSH, SW2 DIPS_04

Commit message: Filled in component details, update board to v1.1
Parts:
- P1: Alt. Order Code (none) -> 855-M20-9991446; Alt. Supplier (none) -> Mouser; Note (none) -> 1x14 header strip; Package (none) -> SIL-14; Supplier (none) -> Farnell
- P2: Alt. Order Code (none) -> ESQ-114-33-G-S; Alt. Supplier (none) -> Samtec; Note (none) -> 1x14 ESQ series elevated socket strip; Package (none) -> SIL-14; Supplier (none) -> Farnell
- P3: Alt. Order Code (none) -> 571-8-188275-4; Alt. Supplier (none) -> Mouser; Note (none) -> 14-way SMD Micro-MaTch connector; Package (none) -> Micro-MaTch SMD 14; Supplier (none) -> Farnell
- P4: Alt. Order Code (none) -> 855-M20-9990445; Alt. Supplier (none) -> Mouser; Note (none) -> 1x4 header strip; Order Code 1926221 -> 1022250; Package (none) -> SIL-4; Part Number HTSW-104-15-G-S -> M20-9990445; Supplier (none) -> Farnell
- P5: Alt. Order Code (none) -> ESQ-104-33-G-S; Alt. Supplier (none) -> Samtec; Note (none) -> 1x4 ESQ series elevated socket strip; Package (none) -> SIL-4; Supplier (none) -> Farnell
- P6: Alt. Order Code (none) -> 523-L77HDE15SD1CH4F; Alt. Supplier (none) -> Mouser; Note (none) -> 15-way D-Sub high density connector; Package (none) -> DSUB15; Supplier (none) -> Farnell
- P7: Alt. Order Code (none) -> 538-95501-2881; Alt. Supplier (none) -> Mouser; Note (none) -> RJ45 8-way R/A jack; Package (none) -> RJ45; Supplier (none) -> Farnell
- R1, R2, R3, R4: Alt. Order Code (none) -> 71-CRCW0805-10K-E3; Alt. Supplier (none) -> Mouser; Note (none) -> 10kΩ/1% 0805 resistor; Package (none) -> 0805; Supplier (none) -> Farnell
- SW1: Alt. Order Code (none) -> 506-FSMRA3JH; Alt. Supplier (none) -> Mouser; Note (none) -> R/A tactile switch; Package (none) -> RA pushbutton; Supplier (none) -> Farnell
- SW2: Alt. Order Code (none) -> 642-DPL04; Alt. Supplier (none) -> Mouser; Note (none) -> 4x vertical SPST DIP switch; Package (none) -> DIL-8; Supplier (none) -> Farnell
Changed lines of the file:
@@
 EESchema Schematic File Version 2
-LIBS:MicroFLiC_I2C_extension_1_0-rescue
 LIBS:power
 LIBS:device
@@
 LIBS:valves
 LIBS:jakub
-LIBS:MicroFLiC_I2C_extension_1_0-cache
+LIBS:MicroFLiC_I2C_extension-cache
 EELAYER 25 0
 EELAYER END
@@
 F 2 "Pin_Headers:Pin_Header_Straight_1x04" H 6850 4450 60  0001 C CNN
 F 3 "" H 6850 4450 60  0000 C CNN
-F 4 "HTSW-104-15-G-S" H 6850 4450 60  0001 C CNN "Part Number"
+F 4 "M20-9990445" H 6850 4450 60  0001 C CNN "Part Number"
 F 5 "Samtec" H 6850 4450 60  0001 C CNN "Manufacturer"
-F 6 "1926221" H 6850 4450 60  0001 C CNN "Order Code"
+F 6 "SIL-4" H 6850 4450 60  0001 C CNN "Package"
+F 7 "Farnell" H 6850 4450 60  0001 C CNN "Supplier"
+F 8 "1022250" H 6850 4450 60  0001 C CNN "Order Code"
+F 9 "Mouser" H 6850 4450 60  0001 C CNN "Alt. Supplier"
+F 10 "855-M20-9990445" H 6850 4450 60  0001 C CNN "Alt. Order Code"
+F 11 "1x4 header strip" H 6850 4450 60  0001 C CNN "Note"
 	1    6850 4450
 	-1   0    0    -1
@@
 F 4 "ESQ-114-33-G-S" H 2500 1950 60  0001 C CNN "Part Number"
 F 5 "Samtec" H 2500 1950 60  0001 C CNN "Manufacturer"
-F 6 "1930609" H 2500 1950 60  0001 C CNN "Order Code"
+F 6 "SIL-14" H 2500 1950 60  0001 C CNN "Package"
+F 7 "Farnell" H 2500 1950 60  0001 C CNN "Supplier"
+F 8 "1930609" H 2500 1950 60  0001 C CNN "Order Code"
+F 9 "Samtec" H 2500 1950 60  0001 C CNN "Alt. Supplier"
+F 10 "ESQ-114-33-G-S" H 2500 1950 60  0001 C CNN "Alt. Order Code"
+F 11 "1x14 ESQ series elevated socket strip" H 2500 1950 60  0001 C CNN "Note"
 	1    2500 1950
 	1    0    0    -1
@@
 F 4 "MC34735" H 1300 1950 60  0001 C CNN "Part Number"
 F 5 "Multicomp" H 1300 1950 60  0001 C CNN "Manufacturer"
-F 6 "1593421" H 1300 1950 60  0001 C CNN "Order Code"
+F 6 "SIL-14" H 1300 1950 60  0001 C CNN "Package"
+F 7 "Farnell" H 1300 1950 60  0001 C CNN "Supplier"
+F 8 "1593421" H 1300 1950 60  0001 C CNN "Order Code"
+F 9 "Mouser" H 1300 1950 60  0001 C CNN "Alt. Supplier"
+F 10 "855-M20-9991446" H 1300 1950 60  0001 C CNN "Alt. Order Code"
+F 11 "1x14 header strip" H 1300 1950 60  0001 C CNN "Note"
 	1    1300 1950
 	-1   0    0    -1
@@
 F 4 "L77HDE15SD1CH4F" H 8900 1950 60  0001 C CNN "Part Number"
 F 5 "Amphenol" H 8900 1950 60  0001 C CNN "Manufacturer"
-F 6 "2401182" H 8900 1950 60  0001 C CNN "Order Code"
+F 6 "DSUB15" H 8900 1950 60  0001 C CNN "Package"
+F 7 "Farnell" H 8900 1950 60  0001 C CNN "Supplier"
+F 8 "2401182" H 8900 1950 60  0001 C CNN "Order Code"
+F 9 "Mouser" H 8900 1950 60  0001 C CNN "Alt. Supplier"
+F 10 "523-L77HDE15SD1CH4F" H 8900 1950 60  0001 C CNN "Alt. Order Code"
+F 11 "15-way D-Sub high density connector" H 8900 1950 60  0001 C CNN "Note"
 	1    8900 1950
 	1    0    0    -1
@@
 F 4 "95501-2881" H 8900 4450 60  0001 C CNN "Part Number"
 F 5 "Molex" H 8900 4450 60  0001 C CNN "Manufacturer"
-F 6 "1524544" H 8900 4450 60  0001 C CNN "Order Code"
+F 6 "RJ45" H 8900 4450 60  0001 C CNN "Package"
+F 7 "Farnell" H 8900 4450 60  0001 C CNN "Supplier"
+F 8 "1524544" H 8900 4450 60  0001 C CNN "Order Code"
+F 9 "Mouser" H 8900 4450 60  0001 C CNN "Alt. Supplier"
+F 10 "538-95501-2881" H 8900 4450 60  0001 C CNN "Alt. Order Code"
+F 11 "RJ45 8-way R/A jack" H 8900 4450 60  0001 C CNN "Note"
 	1    8900 4450
 	0    1    1    0
@@
 F 4 "MCDA04" V 5400 2450 60  0001 C CNN "Part Number"
 F 5 "Multicomp" V 5400 2450 60  0001 C CNN "Manufacturer"
-F 6 "9471545" V 5400 2450 60  0001 C CNN "Order Code"
+F 6 "DIL-8" H 5400 2450 60  0001 C CNN "Package"
+F 7 "Farnell" H 5400 2450 60  0001 C CNN "Supplier"
+F 8 "9471545" V 5400 2450 60  0001 C CNN "Order Code"
+F 9 "Mouser" H 5400 2450 60  0001 C CNN "Alt. Supplier"
+F 10 "642-DPL04" H 5400 2450 60  0001 C CNN "Alt. Order Code"
+F 11 "4x vertical SPST DIP switch" H 5400 2450 60  0001 C CNN "Note"
 	1    5400 2450
 	1    0    0    -1
@@
 F 4 "MCMR08X1002FTL" V 5250 3400 60  0001 C CNN "Part Number"
 F 5 "Multicomp" V 5250 3400 60  0001 C CNN "Manufacturer"
-F 6 "2073607" V 5250 3400 60  0001 C CNN "Order Code"
+F 6 "0805" H 5250 3400 60  0001 C CNN "Package"
+F 7 "Farnell" H 5250 3400 60  0001 C CNN "Supplier"
+F 8 "2073607" V 5250 3400 60  0001 C CNN "Order Code"
+F 9 "Mouser" H 5250 3400 60  0001 C CNN "Alt. Supplier"
+F 10 "71-CRCW0805-10K-E3" H 5250 3400 60  0001 C CNN "Alt. Order Code"
+F 11 "10kΩ/1% 0805 resistor" H 5250 3400 60  0001 C CNN "Note"
 	1    5250 3400
 	1    0    0    -1
@@
 F 4 "MCMR08X1002FTL" V 5350 3400 60  0001 C CNN "Part Number"
 F 5 "Multicomp" V 5350 3400 60  0001 C CNN "Manufacturer"
-F 6 "2073607" V 5350 3400 60  0001 C CNN "Order Code"
+F 6 "0805" H 5350 3400 60  0001 C CNN "Package"
+F 7 "Farnell" H 5350 3400 60  0001 C CNN "Supplier"
+F 8 "2073607" V 5350 3400 60  0001 C CNN "Order Code"
+F 9 "Mouser" H 5350 3400 60  0001 C CNN "Alt. Supplier"
+F 10 "71-CRCW0805-10K-E3" H 5350 3400 60  0001 C CNN "Alt. Order Code"
+F 11 "10kΩ/1% 0805 resistor" H 5350 3400 60  0001 C CNN "Note"
 	1    5350 3400
 	1    0    0    -1
@@
 F 4 "MCMR08X1002FTL" V 5450 3400 60  0001 C CNN "Part Number"
 F 5 "Multicomp" V 5450 3400 60  0001 C CNN "Manufacturer"
-F 6 "2073607" V 5450 3400 60  0001 C CNN "Order Code"
+F 6 "0805" H 5450 3400 60  0001 C CNN "Package"
+F 7 "Farnell" H 5450 3400 60  0001 C CNN "Supplier"
+F 8 "2073607" V 5450 3400 60  0001 C CNN "Order Code"
+F 9 "Mouser" H 5450 3400 60  0001 C CNN "Alt. Supplier"
+F 10 "71-CRCW0805-10K-E3" H 5450 3400 60  0001 C CNN "Alt. Order Code"
+F 11 "10kΩ/1% 0805 resistor" H 5450 3400 60  0001 C CNN "Note"
 	1    5450 3400
 	1    0    0    -1
@@
 F 4 "MCMR08X1002FTL" V 5550 3400 60  0001 C CNN "Part Number"
 F 5 "Multicomp" V 5550 3400 60  0001 C CNN "Manufacturer"
-F 6 "2073607" V 5550 3400 60  0001 C CNN "Order Code"
+F 6 "0805" H 5550 3400 60  0001 C CNN "Package"
+F 7 "Farnell" H 5550 3400 60  0001 C CNN "Supplier"
+F 8 "2073607" V 5550 3400 60  0001 C CNN "Order Code"
+F 9 "Mouser" H 5550 3400 60  0001 C CNN "Alt. Supplier"
+F 10 "71-CRCW0805-10K-E3" H 5550 3400 60  0001 C CNN "Alt. Order Code"
+F 11 "10kΩ/1% 0805 resistor" H 5550 3400 60  0001 C CNN "Note"
 	1    5550 3400
 	1    0    0    -1
@@
 F 4 "MCDTSA6-5N" H 3600 4500 60  0001 C CNN "Part Number"
 F 5 "Multicomp" H 3600 4500 60  0001 C CNN "Manufacturer"
-F 6 "9471804" H 3600 4500 60  0001 C CNN "Order Code"
+F 6 "RA pushbutton" H 3600 4500 60  0001 C CNN "Package"
+F 7 "Farnell" H 3600 4500 60  0001 C CNN "Supplier"
+F 8 "9471804" H 3600 4500 60  0001 C CNN "Order Code"
+F 9 "Mouser" H 3600 4500 60  0001 C CNN "Alt. Supplier"
+F 10 "506-FSMRA3JH" H 3600 4500 60  0001 C CNN "Alt. Order Code"
+F 11 "R/A tactile switch" H 3600 4500 60  0001 C CNN "Note"
 	1    3600 4500
 	1    0    0    -1
@@
 F 4 "8-188275-4" H 2600 4400 60  0001 C CNN "Part Number"
 F 5 "TE Connectivity" H 2600 4400 60  0001 C CNN "Manufacturer"
-F 6 "3784769" H 2600 4400 60  0001 C CNN "Order Code"
+F 6 "Micro-MaTch SMD 14" H 2600 4400 60  0001 C CNN "Package"
+F 7 "Farnell" H 2600 4400 60  0001 C CNN "Supplier"
+F 8 "3784769" H 2600 4400 60  0001 C CNN "Order Code"
+F 9 "Mouser" H 2600 4400 60  0001 C CNN "Alt. Supplier"
+F 10 "571-8-188275-4" H 2600 4400 60  0001 C CNN "Alt. Order Code"
+F 11 "14-way SMD Micro-MaTch connector" H 2600 4400 60  0001 C CNN "Note"
 	1    2600 4400
 	1    0    0    -1
@@
 F 4 "ESQ-104-33-G-S" H 6850 5100 60  0001 C CNN "Part Number"
 F 5 "Samtec" H 6850 5100 60  0001 C CNN "Manufacturer"
-F 6 "1928522" H 6850 5100 60  0001 C CNN "Order Code"
+F 6 "SIL-4" H 6850 5100 60  0001 C CNN "Package"
+F 7 "Farnell" H 6850 5100 60  0001 C CNN "Supplier"
+F 8 "1928522" H 6850 5100 60  0001 C CNN "Order Code"
+F 9 "Samtec" H 6850 5100 60  0001 C CNN "Alt. Supplier"
+F 10 "ESQ-104-33-G-S" H 6850 5100 60  0001 C CNN "Alt. Order Code"
+F 11 "1x4 ESQ series elevated socket strip" H 6850 5100 60  0001 C CNN "Note"
 	1    6850 5100
 	-1   0    0    -1

Commit message: Fixed connector descriptions
Parts:
- P1: value Header_1x14 -> 1x14 header strip
- P2: value Socket_1x14 -> 1x14 socket strip
- P3: value Micro-MaTch 14 way -> 14-way Micro-MaTch
- P4: value Header_1x4 -> 1x4 header strip
- P5: value Socket_1x4 -> 1x4 socket strip
- SW1: value SW_PUSH -> Tactile switch R/A
Other:
- moved on the sheet: P4, P5, P7
Changed lines of the file:
@@
 L CONN_01X04 P4
 U 1 1 54DF35DA
-P 6850 4450
-F 0 "P4" H 6850 4700 50  0000 C CNN
-F 1 "Header_1x4" V 6950 4450 50  0000 C CNN
-F 2 "Pin_Headers:Pin_Header_Straight_1x04" H 6850 4450 60  0001 C CNN
-F 3 "" H 6850 4450 60  0000 C CNN
-F 4 "M20-9990445" H 6850 4450 60  0001 C CNN "Part Number"
-F 5 "Samtec" H 6850 4450 60  0001 C CNN "Manufacturer"
-F 6 "SIL-4" H 6850 4450 60  0001 C CNN "Package"
-F 7 "Farnell" H 6850 4450 60  0001 C CNN "Supplier"
-F 8 "1022250" H 6850 4450 60  0001 C CNN "Order Code"
-F 9 "Mouser" H 6850 4450 60  0001 C CNN "Alt. Supplier"
-F 10 "855-M20-9990445" H 6850 4450 60  0001 C CNN "Alt. Order Code"
-F 11 "1x4 header strip" H 6850 4450 60  0001 C CNN "Note"
-	1    6850 4450
+P 6800 4450
+F 0 "P4" H 6800 4700 50  0000 C CNN
+F 1 "1x4 header strip" V 6900 4450 50  0000 C CNN
+F 2 "Pin_Headers:Pin_Header_Straight_1x04" H 6800 4450 60  0001 C CNN
+F 3 "" H 6800 4450 60  0000 C CNN
+F 4 "M20-9990445" H 6800 4450 60  0001 C CNN "Part Number"
+F 5 "Samtec" H 6800 4450 60  0001 C CNN "Manufacturer"
+F 6 "SIL-4" H 6800 4450 60  0001 C CNN "Package"
+F 7 "Farnell" H 6800 4450 60  0001 C CNN "Supplier"
+F 8 "1022250" H 6800 4450 60  0001 C CNN "Order Code"
+F 9 "Mouser" H 6800 4450 60  0001 C CNN "Alt. Supplier"
+F 10 "855-M20-9990445" H 6800 4450 60  0001 C CNN "Alt. Order Code"
+F 11 "1x4 header strip" H 6800 4450 60  0001 C CNN "Note"
+	1    6800 4450
 	-1   0    0    -1
 $EndComp
@@
 P 2500 1950
 F 0 "P2" H 2500 2700 50  0000 C CNN
-F 1 "Socket_1x14" V 2600 1950 50  0000 C CNN
+F 1 "1x14 socket strip" V 2600 1950 50  0000 C CNN
 F 2 "jakub:ESQ-114-33-G-S" H 2500 1950 60  0001 C CNN
 F 3 "" H 2500 1950 60  0000 C CNN
@@
 P 1300 1950
 F 0 "P1" H 1300 2700 50  0000 C CNN
-F 1 "Header_1x14" V 1400 1950 50  0000 C CNN
+F 1 "1x14 header strip" V 1400 1950 50  0000 C CNN
 F 2 "Pin_Headers:Pin_Header_Straight_1x14" H 1300 1950 60  0001 C CNN
 F 3 "" H 1300 1950 60  0000 C CNN
@@
 $EndComp
 Wire Wire Line
-	7050 4300 8000 4300
-Wire Wire Line
-	7050 4400 8450 4400
+	7000 4300 8000 4300
+Wire Wire Line
+	7000 4400 8500 4400
 Wire Wire Line
 	2350 4600 1900 4600
@@
 	2350 4200 1900 4200
 Wire Wire Line
-	7050 4500 8450 4500
-Wire Wire Line
-	7050 4600 8000 4600
+	7000 4500 8500 4500
+Wire Wire Line
+	7000 4600 8000 4600
 Wire Wire Line
 	1500 1300 2300 1300
@@
 L RJ45 P7
 U 1 1 556B8802
-P 8900 4450
-F 0 "P7" H 9100 4950 60  0000 C CNN
-F 1 "RJ45" H 8750 4950 60  0000 C CNN
-F 2 "jakub:RJ45" H 8900 4450 60  0001 C CNN
-F 3 "" H 8900 4450 60  0000 C CNN
-F 4 "95501-2881" H 8900 4450 60  0001 C CNN "Part Number"
-F 5 "Molex" H 8900 4450 60  0001 C CNN "Manufacturer"
-F 6 "RJ45" H 8900 4450 60  0001 C CNN "Package"
-F 7 "Farnell" H 8900 4450 60  0001 C CNN "Supplier"
-F 8 "1524544" H 8900 4450 60  0001 C CNN "Order Code"
-F 9 "Mouser" H 8900 4450 60  0001 C CNN "Alt. Supplier"
-F 10 "538-95501-2881" H 8900 4450 60  0001 C CNN "Alt. Order Code"
-F 11 "RJ45 8-way R/A jack" H 8900 4450 60  0001 C CNN "Note"
-	1    8900 4450
+P 8950 4450
+F 0 "P7" H 9150 4950 60  0000 C CNN
+F 1 "RJ45" H 8800 4950 60  0000 C CNN
+F 2 "jakub:RJ45" H 8950 4450 60  0001 C CNN
+F 3 "" H 8950 4450 60  0000 C CNN
+F 4 "95501-2881" H 8950 4450 60  0001 C CNN "Part Number"
+F 5 "Molex" H 8950 4450 60  0001 C CNN "Manufacturer"
+F 6 "RJ45" H 8950 4450 60  0001 C CNN "Package"
+F 7 "Farnell" H 8950 4450 60  0001 C CNN "Supplier"
+F 8 "1524544" H 8950 4450 60  0001 C CNN "Order Code"
+F 9 "Mouser" H 8950 4450 60  0001 C CNN "Alt. Supplier"
+F 10 "538-95501-2881" H 8950 4450 60  0001 C CNN "Alt. Order Code"
+F 11 "RJ45 8-way R/A jack" H 8950 4450 60  0001 C CNN "Note"
+	1    8950 4450
 	0    1    1    0
 $EndComp
 Wire Wire Line
-	8450 4200 8000 4200
+	8500 4200 8000 4200
 Wire Wire Line
 	8000 4200 8000 4300
@@
 	8000 4600 8000 4700
 Wire Wire Line
-	8000 4700 8450 4700
-Wire Wire Line
-	8450 4300 8350 4300
-Wire Wire Line
-	8350 4300 8350 5000
-Wire Wire Line
-	8450 4800 8350 4800
-Connection ~ 8350 4800
-Wire Wire Line
-	8450 4600 8150 4600
-Wire Wire Line
-	8150 4600 8150 4100
-Wire Wire Line
-	8450 4100 8350 4100
-Wire Wire Line
-	8350 4100 8350 3900
+	8000 4700 8500 4700
+Wire Wire Line
+	8500 4300 8400 4300
+Wire Wire Line
+	8400 4300 8400 5000
+Wire Wire Line
+	8500 4800 8400 4800
+Connection ~ 8400 4800
+Wire Wire Line
+	8500 4600 8200 4600
+Wire Wire Line
+	8200 4600 8200 4100
+Wire Wire Line
+	8500 4100 8400 4100
+Wire Wire Line
+	8400 4100 8400 3900
 $Comp
 L +5VP #PWR06
 U 1 1 556B9C52
-P 8350 3900
-F 0 "#PWR06" H 8350 3750 60  0001 C CNN
-F 1 "+5VP" H 8350 4040 60  0000 C CNN
-F 2 "" H 8350 3900 60  0000 C CNN
-F 3 "" H 8350 3900 60  0000 C CNN
-	1    8350 3900
+P 8400 3900
+F 0 "#PWR06" H 8400 3750 60  0001 C CNN
+F 1 "+5VP" H 8400 4040 60  0000 C CNN
+F 2 "" H 8400 3900 60  0000 C CNN
+F 3 "" H 8400 3900 60  0000 C CNN
+	1    8400 3900
 	1    0    0    -1
 $EndComp
@@
 L +3V3 #PWR07
 U 1 1 556B9C72
-P 8150 4100
-F 0 "#PWR07" H 8150 3950 60  0001 C CNN
-F 1 "+3V3" H 8150 4240 60  0000 C CNN
-F 2 "" H 8150 4100 60  0000 C CNN
-F 3 "" H 8150 4100 60  0000 C CNN
-	1    8150 4100
+P 8200 4100
+F 0 "#PWR07" H 8200 3950 60  0001 C CNN
+F 1 "+3V3" H 8200 4240 60  0000 C CNN
+F 2 "" H 8200 4100 60  0000 C CNN
+F 3 "" H 8200 4100 60  0000 C CNN
+	1    8200 4100
 	1    0    0    -1
 $EndComp
@@
 L GND #PWR08
 U 1 1 556B9CAA
-P 8350 5000
-F 0 "#PWR08" H 8350 4750 60  0001 C CNN
-F 1 "GND" H 8350 4850 60  0000 C CNN
-F 2 "" H 8350 5000 60  0000 C CNN
-F 3 "" H 8350 5000 60  0000 C CNN
-	1    8350 5000
+P 8400 5000
+F 0 "#PWR08" H 8400 4750 60  0001 C CNN
+F 1 "GND" H 8400 4850 60  0000 C CNN
+F 2 "" H 8400 5000 60  0000 C CNN
+F 3 "" H 8400 5000 60  0000 C CNN
+	1    8400 5000
 	1    0    0    -1
 $EndComp
@@
 P 3600 4500
 F 0 "SW1" H 3750 4610 50  0000 C CNN
-F 1 "SW_PUSH" H 3600 4420 50  0000 C CNN
+F 1 "Tactile switch R/A" H 3600 4420 50  0000 C CNN
 F 2 "jakub:tactileSwitchRA" H 3600 4500 60  0001 C CNN
 F 3 "" H 3600 4500 60  0000 C CNN
@@
 P 2600 4400
 F 0 "P3" H 2600 4800 50  0000 C CNN
-F 1 "Micro-MaTch 14 way" H 2600 4000 50  0000 C CNN
+F 1 "14-way Micro-MaTch" H 2600 4000 50  0000 C CNN
 F 2 "jakub:1-188275-4" H 2600 3200 60  0001 C CNN
 F 3 "" H 2600 3200 60  0000 C CNN
@@
 Wire Wire Line
 	2350 4700 1900 4700
-NoConn ~ 9250 5000
+NoConn ~ 9300 5000
 Wire Wire Line
 	8350 2850 8250 2850
@@
 L CONN_01X04 P5
 U 1 1 55C2BA8F
-P 6850 5100
-F 0 "P5" H 6850 5350 50  0000 C CNN
-F 1 "Socket_1x4" V 6950 5100 50  0000 C CNN
-F 2 "jakub:ESQ-104-33-G-S" H 6850 5100 60  0001 C CNN
-F 3 "" H 6850 5100 60  0000 C CNN
-F 4 "ESQ-104-33-G-S" H 6850 5100 60  0001 C CNN "Part Number"
-F 5 "Samtec" H 6850 5100 60  0001 C CNN "Manufacturer"
-F 6 "SIL-4" H 6850 5100 60  0001 C CNN "Package"
-F 7 "Farnell" H 6850 5100 60  0001 C CNN "Supplier"
-F 8 "1928522" H 6850 5100 60  0001 C CNN "Order Code"
-F 9 "Samtec" H 6850 5100 60  0001 C CNN "Alt. Supplier"
-F 10 "ESQ-104-33-G-S" H 6850 5100 60  0001 C CNN "Alt. Order Code"
-F 11 "1x4 ESQ series elevated socket strip" H 6850 5100 60  0001 C CNN "Note"
-	1    6850 5100
+P 6800 5150
+F 0 "P5" H 6800 5400 50  0000 C CNN
+F 1 "1x4 socket strip" V 6900 5150 50  0000 C CNN
+F 2 "jakub:ESQ-104-33-G-S" H 6800 5150 60  0001 C CNN
+F 3 "" H 6800 5150 60  0000 C CNN
+F 4 "ESQ-104-33-G-S" H 6800 5150 60  0001 C CNN "Part Number"
+F 5 "Samtec" H 6800 5150 60  0001 C CNN "Manufacturer"
+F 6 "SIL-4" H 6800 5150 60  0001 C CNN "Package"
+F 7 "Farnell" H 6800 5150 60  0001 C CNN "Supplier"
+F 8 "1928522" H 6800 5150 60  0001 C CNN "Order Code"
+F 9 "Samtec" H 6800 5150 60  0001 C CNN "Alt. Supplier"
+F 10 "ESQ-104-33-G-S" H 6800 5150 60  0001 C CNN "Alt. Order Code"
+F 11 "1x4 ESQ series elevated socket strip" H 6800 5150 60  0001 C CNN "Note"
+	1    6800 5150
 	-1   0    0    -1
 $EndComp
 Wire Wire Line
-	7050 4950 7600 4950
-Wire Wire Line
-	7600 4950 7600 4300
+	7000 5000 7600 5000
+Wire Wire Line
+	7600 5000 7600 4300
 Connection ~ 7600 4300
 Wire Wire Line
-	7700 4400 7700 5050
-Wire Wire Line
-	7700 5050 7050 5050
+	7700 4400 7700 5100
+Wire Wire Line
+	7700 5100 7000 5100
 Connection ~ 7700 4400
 Wire Wire Line
-	7050 5150 7800 5150
-Wire Wire Line
-	7800 5150 7800 4500
+	7000 5200 7800 5200
+Wire Wire Line
+	7800 5200 7800 4500
 Connection ~ 7800 4500
 Wire Wire Line
-	7900 4600 7900 5250
-Wire Wire Line
-	7900 5250 7050 5250
+	7900 4600 7900 5300
+Wire Wire Line
+	7900 5300 7000 5300
 Connection ~ 7900 4600
 $EndSCHEMATC

Commit message: Minor part description changes
Parts:
- P4: Manufacturer Samtec -> Harwin
- SW1: Note R/A tactile switch -> Right-angle tactile switch; Package RA pushbutton -> R/A pushbutton
Changed lines of the file:
@@
 F 3 "" H 6800 4450 60  0000 C CNN
 F 4 "M20-9990445" H 6800 4450 60  0001 C CNN "Part Number"
-F 5 "Samtec" H 6800 4450 60  0001 C CNN "Manufacturer"
+F 5 "Harwin" H 6800 4450 60  0001 C CNN "Manufacturer"
 F 6 "SIL-4" H 6800 4450 60  0001 C CNN "Package"
 F 7 "Farnell" H 6800 4450 60  0001 C CNN "Supplier"
@@
 F 4 "MCDTSA6-5N" H 3600 4500 60  0001 C CNN "Part Number"
 F 5 "Multicomp" H 3600 4500 60  0001 C CNN "Manufacturer"
-F 6 "RA pushbutton" H 3600 4500 60  0001 C CNN "Package"
+F 6 "R/A pushbutton" H 3600 4500 60  0001 C CNN "Package"
 F 7 "Farnell" H 3600 4500 60  0001 C CNN "Supplier"
 F 8 "9471804" H 3600 4500 60  0001 C CNN "Order Code"
 F 9 "Mouser" H 3600 4500 60  0001 C CNN "Alt. Supplier"
 F 10 "506-FSMRA3JH" H 3600 4500 60  0001 C CNN "Alt. Order Code"
-F 11 "R/A tactile switch" H 3600 4500 60  0001 C CNN "Note"
+F 11 "Right-angle tactile switch" H 3600 4500 60  0001 C CNN "Note"
 	1    3600 4500
 	1    0    0    -1
